Commit message: update path to ros2 format

File: realsense2_description/urdf/_d415.urdf.xacro (robot description, xacro)
@@ -46,5 +46,5 @@
           <origin xyz="${d415_cam_mount_from_center_offset} ${-d415_cam_depth_py} 0" rpy="${M_PI/2} 0 ${M_PI/2}"/>
           <geometry>
-            <mesh filename="package://realsense2_description/meshes/d415.stl" />
+            <mesh filename="$(find realsense2_description)/meshes/d415.stl" />
           </geometry>
           <material name="aluminum"/>

File: realsense2_description/urdf/_d455.urdf.xacro (robot description, xacro)
@@ -55,5 +55,5 @@
         <geometry>
           <!-- <box size="${d455_cam_depth} ${d455_cam_width} ${d455_cam_height}"/> -->
-	        <mesh filename="package://realsense2_description/meshes/d455.stl" scale="0.001 0.001 0.001" />
+	        <mesh filename="$(find realsense2_description)/meshes/d455.stl" scale="0.001 0.001 0.001" />
         </geometry>
         <material name="aluminum"/>

File: realsense2_description/urdf/_l515.urdf.xacro (robot description, xacro)
@@ -63,5 +63,5 @@
           <origin xyz="${l515_zero_depth_to_glass} 0 ${-l515_cam_center_to_depth_pz}" rpy="${M_PI/2} 0 ${M_PI/2}"/>
           <geometry>
-              <mesh filename="package://realsense2_description/meshes/l515.dae" />
+              <mesh filename="$(find realsense2_description)/realsense2_description/meshes/l515.dae" />
           </geometry>
         </xacro:if>

File: realsense2_description/urdf/_r410.urdf.xacro (robot description, xacro)
@@ -38,5 +38,5 @@
         <geometry>
           <box size="${r410_cam_width} ${r410_cam_height} ${r410_cam_depth}"/>
-          <!--<mesh filename="package://realsense2_description/meshes/r410/r410.dae" />-->
+          <!--<mesh filename="$(find realsense2_description)/meshes/r410/r410.dae" />-->
         </geometry>
         <material name="aluminum"/>

File: realsense2_description/urdf/_r430.urdf.xacro (robot description, xacro)
@@ -39,5 +39,5 @@
         <geometry>
           <box size="${r430_cam_width} ${r430_cam_height} ${r430_cam_depth}"/>
-          <!--<mesh filename="package://realsense2_description/meshes/r430/r430.dae" />-->
+          <!--<mesh filename="$(find realsense2_description)/meshes/r430/r430.dae" />-->
         </geometry>
         <material name="aluminum"/>

File: realsense2_description/urdf/_usb_plug.urdf.xacro (robot description, xacro)
@@ -20,5 +20,5 @@
         <geometry>
           <!--box size="0.044850 0.008 0.0185" /-->
-          <mesh filename="package://realsense2_description/meshes/plug.stl" />
+          <mesh filename="$(find realsense2_description)/meshes/plug.stl" />
         </geometry>
         <material name="plastic"/>
@@ -28,5 +28,5 @@
         <geometry>
           <!--box size="0.044850 0.008 0.0185" /-->
-          <mesh filename="package://realsense2_description/meshes/plug_collision.stl" />
+          <mesh filename="$(find realsense2_description)/meshes/plug_collision.stl" />
         </geometry>
       </collision>
