Commit message: update urdf to gazebo support

File: realsense2_description/urdf/_d435.urdf.xacro (robot description, xacro)
@@ -10,5 +10,6 @@
   <xacro:include filename="$(find realsense2_description)/urdf/_materials.urdf.xacro" />
   <xacro:include filename="$(find realsense2_description)/urdf/_usb_plug.urdf.xacro" />
-  <xacro:macro name="sensor_d435" params="parent *origin name:=camera use_nominal_extrinsics:=false add_plug:=false use_mesh:=true">
+  <xacro:include filename="$(find realsense2_description)/urdf/_d435.gazebo.xacro"/>
+  <xacro:macro name="sensor_d435" params="parent *origin name:=camera use_nominal_extrinsics:=false add_plug:=false use_mesh:=true topics_ns:=camera publish_pointcloud:=true">
     <xacro:property name="M_PI" value="3.1415926535897931" />
     <!-- The following values are approximate, and the camera node
@@ -137,4 +138,5 @@
       </xacro:usb_plug>
     </xacro:if>
+    <xacro:gazebo_d435 camera_name="${name}" reference_link="${name}_link" topics_ns="${topics_ns}" depth_optical_frame="${name}_depth_optical_frame" color_optical_frame="${name}_color_optical_frame" infrared1_optical_frame="${name}_left_ir_optical_frame" infrared2_optical_frame="${name}_right_ir_optical_frame" publish_pointcloud="${publish_pointcloud}"/>
   </xacro:macro>
 </robot>

Commit message: update path to ros2 format

File: realsense2_description/urdf/_d435.urdf.xacro (robot description, xacro)
@@ -54,5 +54,5 @@
           <origin xyz="${d435_zero_depth_to_glass + d435_glass_to_front} ${-d435_cam_depth_py} 0" rpy="${M_PI/2} 0 ${M_PI/2}"/>
           <geometry>
-            <mesh filename="package://realsense2_description/meshes/d435.dae" />
+            <mesh filename="$(find realsense2_description)/meshes/d435.dae" />
           </geometry>
         </xacro:if>

Commit message: update path for ros2

File: realsense2_description/urdf/_d435.urdf.xacro (robot description, xacro)
@@ -54,5 +54,5 @@
           <origin xyz="${d435_zero_depth_to_glass + d435_glass_to_front} ${-d435_cam_depth_py} 0" rpy="${M_PI/2} 0 ${M_PI/2}"/>
           <geometry>
-            <mesh filename="$(find realsense2_description)/meshes/d435.dae" />
+            <mesh filename="file://$(find realsense2_description)/meshes/d435.dae" />
           </geometry>
         </xacro:if>

File: realsense2_description/urdf/_usb_plug.urdf.xacro (robot description, xacro)
@@ -20,5 +20,5 @@
         <geometry>
           <!--box size="0.044850 0.008 0.0185" /-->
-          <mesh filename="$(find realsense2_description)/meshes/plug.stl" />
+          <mesh filename="file://$(find realsense2_description)/meshes/plug.stl" />
         </geometry>
         <material name="plastic"/>
@@ -28,5 +28,5 @@
         <geometry>
           <!--box size="0.044850 0.008 0.0185" /-->
-          <mesh filename="$(find realsense2_description)/meshes/plug_collision.stl" />
+          <mesh filename="file://$(find realsense2_description)/meshes/plug_collision.stl" />
         </geometry>
       </collision>
